File: pcb/FP2800A-Tester.kicad_sch (KiCad schematic)
At the start: 4 parts, among them SW1 Reset, U1 FP2800A

Commit message: style: add variables
Other:
- title: (none) -> FP2800A-Tester
Changed lines of the file:
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@@
 (kicad_sch (version 20230121) (generator eeschema)
   (paper "A4")
+  (title_block
+    (title "FP2800A-Tester")
+    (date "${DATE}")
+    (rev "${VERSION}")
+  )
   (junction (at 154.94 93.98) (diameter 0) (color 0 0 0 0)
   )

Commit message: feat: add part numbers for production
Parts:
- C1: LCSC (none) -> C14663
Changed lines of the file:
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@@
+      (effects (font (size 1.27 1.27)) hide)
+    )
+    (property "LCSC" "" (at 66.04 60.96 0)
       (effects (font (size 1.27 1.27)) hide)
     )
@@
       (effects (font (size 1.27 1.27)) hide)
     )
+    (property "LCSC" "" (at 43.18 45.72 0)
+      (effects (font (size 1.27 1.27)) hide)
+    )
     (pin "1")
     (pin "2")
@@
     )
     (property "Datasheet" "~" (at 107.95 45.72 0)
+      (effects (font (size 1.27 1.27)) hide)
+    )
+    (property "LCSC" "C14663" (at 107.95 45.72 0)
       (effects (font (size 1.27 1.27)) hide)
     )
@@
       (effects (font (size 1.27 1.27)) hide)
     )
+    (property "LCSC" "" (at 115.57 45.72 0)
+      (effects (font (size 1.27 1.27)) hide)
+    )
